File: Hardware/DC32_Cassette_SAO/DC32_Cassette_SAO.kicad_pcb (KiCad board)
At the start: 2 copper layers, 64.5 x 40.9 mm, 19 parts, among them J1 Conn_02x03_Top_Bottom

Commit message: PCB updates
Parts:
- removed the G*** at (150.0, 100.0)
- added G***: LOGO, DC32_Cassette_SAO:Cassette_SAO_Silk_Screen with Text, F.Cu at (150.0, 100.0)
- moved R1 34.3 mm to (154.6, 118.0), turned to 180 degrees
Routing:
- net Net-(J1-Pin_6): track 6.93 -> 73.1 mm
- net GND: track 151.4 -> 152.6 mm
